File: fonte_3v_12v.brd (EAGLE design)
At the start: 100 x 80 mm, 15 parts, among them IC1 7812TV

Commit message: Add files via upload
Parts:
- removed CAP2: (no value), rcl:E5-13
- removed R3: (no value), rcl:0204/7
- moved TRANSFORMADOR 27.8 mm to (64.3, 55.0)
- moved JP3 23.1 mm to (70.5, 46.2)
- moved CAP3 22.5 mm to (84.6, 23.4)
- moved D1 20.8 mm to (29.3, 51.3), turned to 180 degrees
- moved IC1 19.4 mm to (43.4, 62.0), turned to 90 degrees
- moved CAP4 13.7 mm to (18.4, 23.5)
- moved BRIDGE 13.7 mm to (41.9, 40.3)
- moved R2 12.3 mm to (91.1, 43.2)
- moved D2 10.8 mm to (26.9, 58.8), turned to 0 degrees
- moved CAP1 9.92 mm to (49.9, 7.49)
- moved R1 8.89 mm to (33.7, 72.5)
- moved R4 8.57 mm to (85.5, 60.3)
- moved JP2 4.52 mm to (91.6, 74.8)
Connections:
- removed net N$10: BRIDGE.+, CAP1.+, R3.2
- net N$3: no longer R3.1
- net N$5: now also BRIDGE.+, CAP1.+; no longer CAP2.+
- net N$8: no longer CAP2.-
Routing:
- net N$10: track 74.5 -> 0.00 mm
- net N$5: track 157.3 -> 84.1 mm
- net N$3: track 148.8 -> 127.6 mm
- net N$9: track 84.1 -> 97.8 mm
- net N$4: track 14.6 -> 27.4 mm
- net N$6: track 6.54 -> 15.3 mm
- net N$2: track 23.3 -> 20.7 mm
- net N$8: track 164.2 -> 165.6 mm
- net N$1: track 12.2 -> 11.1 mm
